File: silkscreen-light-strip.kicad_sch (KiCad schematic)
At the start: 18 parts, among them J1 FPC tail to J3

Commit message: Fabrication Toolkit support: rotation-offset fields, pinned coverlay margin, preset layers
Every placed part already had an LCSC field. D13/D14 now also carry
FT Rotation Offset = 180 (LEDs 0), from params, so the toolkit's
placement file matches jlc_cpl.csv. Each footprint pins its coverlay
opening at the 0.1 mm mask expansion, so a plotter that changes the
board-wide margin can't shrink it. fabrication-toolkit-options.json
adds the stiffener and adhesive layers (User.1, User.2), keeps the
bend zones out and names the outputs apart from production/bom.csv.
Gerbers and drill are geometrically unchanged.
Parts:
- D1, D10, D11, D12, D2, D3, D4, D5, D6, D7, D8, D9: FT Rotation Offset (none) -> 0
- D13, D14: FT Rotation Offset (none) -> 180
Changed lines of the file:
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@@
 		(property "Manufacturer" "Nexperia" (at 83.82 40.64 0) (effects (font (size 1.27 1.27)) (hide yes)))
 		(property "LCSC" "C28064" (at 83.82 40.64 0) (effects (font (size 1.27 1.27)) (hide yes)))
+		(property "FT Rotation Offset" "180" (at 83.82 40.64 0) (effects (font (size 1.27 1.27)) (hide yes)))
 		(pin "1")
 		(pin "2")
@@
 		(property "Manufacturer" "XINGLIGHT" (at 109.22 55.88 0) (effects (font (size 1.27 1.27)) (hide yes)))
 		(property "LCSC" "C5440667" (at 109.22 55.88 0) (effects (font (size 1.27 1.27)) (hide yes)))
+		(property "FT Rotation Offset" "0" (at 109.22 55.88 0) (effects (font (size 1.27 1.27)) (hide yes)))
 		(pin "1")
 		(pin "2")
@@
 		(property "Manufacturer" "XINGLIGHT" (at 127 55.88 0) (effects (font (size 1.27 1.27)) (hide yes)))
 		(property "LCSC" "C5440667" (at 127 55.88 0) (effects (font (size 1.27 1.27)) (hide yes)))
+		(property "FT Rotation Offset" "0" (at 127 55.88 0) (effects (font (size 1.27 1.27)) (hide yes)))
 		(pin "1")
 		(pin "2")
@@
 		(property "Manufacturer" "XINGLIGHT" (at 144.78 55.88 0) (effects (font (size 1.27 1.27)) (hide yes)))
 		(property "LCSC" "C5440667" (at 144.78 55.88 0) (effects (font (size 1.27 1.27)) (hide yes)))
+		(property "FT Rotation Offset" "0" (at 144.78 55.88 0) (effects (font (size 1.27 1.27)) (hide yes)))
 		(pin "1")
 		(pin "2")
@@
 		(property "Manufacturer" "XINGLIGHT" (at 162.56 55.88 0) (effects (font (size 1.27 1.27)) (hide yes)))
 		(property "LCSC" "C5440667" (at 162.56 55.88 0) (effects (font (size 1.27 1.27)) (hide yes)))
+		(property "FT Rotation Offset" "0" (at 162.56 55.88 0) (effects (font (size 1.27 1.27)) (hide yes)))
 		(pin "1")
 		(pin "2")
@@
 		(property "Manufacturer" "XINGLIGHT" (at 180.34 55.88 0) (effects (font (size 1.27 1.27)) (hide yes)))
 		(property "LCSC" "C5440667" (at 180.34 55.88 0) (effects (font (size 1.27 1.27)) (hide yes)))
+		(property "FT Rotation Offset" "0" (at 180.34 55.88 0) (effects (font (size 1.27 1.27)) (hide yes)))
 		(pin "1")
 		(pin "2")
@@
 		(property "Manufacturer" "XINGLIGHT" (at 198.12 55.88 0) (effects (font (size 1.27 1.27)) (hide yes)))
 		(property "LCSC" "C5440667" (at 198.12 55.88 0) (effects (font (size 1.27 1.27)) (hide yes)))
+		(property "FT Rotation Offset" "0" (at 198.12 55.88 0) (effects (font (size 1.27 1.27)) (hide yes)))
 		(pin "1")
 		(pin "2")
@@
 		(property "Manufacturer" "Nexperia" (at 83.82 86.36 0) (effects (font (size 1.27 1.27)) (hide yes)))
 		(property "LCSC" "C28064" (at 83.82 86.36 0) (effects (font (size 1.27 1.27)) (hide yes)))
+		(property "FT Rotation Offset" "180" (at 83.82 86.36 0) (effects (font (size 1.27 1.27)) (hide yes)))
 		(pin "1")
 		(pin "2")
@@
 		(property "Manufacturer" "XINGLIGHT" (at 109.22 101.6 0) (effects (font (size 1.27 1.27)) (hide yes)))
 		(property "LCSC" "C2843774" (at 109.22 101.6 0) (effects (font (size 1.27 1.27)) (hide yes)))
+		(property "FT Rotation Offset" "0" (at 109.22 101.6 0) (effects (font (size 1.27 1.27)) (hide yes)))
 		(pin "1")
 		(pin "2")
@@
 		(property "Manufacturer" "XINGLIGHT" (at 127 101.6 0) (effects (font (size 1.27 1.27)) (hide yes)))
 		(property "LCSC" "C2843774" (at 127 101.6 0) (effects (font (size 1.27 1.27)) (hide yes)))
+		(property "FT Rotation Offset" "0" (at 127 101.6 0) (effects (font (size 1.27 1.27)) (hide yes)))
 		(pin "1")
 		(pin "2")
@@
 		(property "Manufacturer" "XINGLIGHT" (at 144.78 101.6 0) (effects (font (size 1.27 1.27)) (hide yes)))
 		(property "LCSC" "C2843774" (at 144.78 101.6 0) (effects (font (size 1.27 1.27)) (hide yes)))
+		(property "FT Rotation Offset" "0" (at 144.78 101.6 0) (effects (font (size 1.27 1.27)) (hide yes)))
 		(pin "1")
 		(pin "2")
@@
 		(property "Manufacturer" "XINGLIGHT" (at 162.56 101.6 0) (effects (font (size 1.27 1.27)) (hide yes)))
 		(property "LCSC" "C2843774" (at 162.56 101.6 0) (effects (font (size 1.27 1.27)) (hide yes)))
+		(property "FT Rotation Offset" "0" (at 162.56 101.6 0) (effects (font (size 1.27 1.27)) (hide yes)))
 		(pin "1")
 		(pin "2")
@@
 		(property "Manufacturer" "XINGLIGHT" (at 180.34 101.6 0) (effects (font (size 1.27 1.27)) (hide yes)))
 		(property "LCSC" "C2843774" (at 180.34 101.6 0) (effects (font (size 1.27 1.27)) (hide yes)))
+		(property "FT Rotation Offset" "0" (at 180.34 101.6 0) (effects (font (size 1.27 1.27)) (hide yes)))
 		(pin "1")
 		(pin "2")
@@
 		(property "Manufacturer" "XINGLIGHT" (at 198.12 101.6 0) (effects (font (size 1.27 1.27)) (hide yes)))
 		(property "LCSC" "C2843774" (at 198.12 101.6 0) (effects (font (size 1.27 1.27)) (hide yes)))
-		(pin "1")
-		(pin "2")
+		(property "FT Rotation Offset" "0" (at 198.12 101.6 0) (effects (font (size 1.27 1.27)) (hide yes)))
+		(pin "1")
+		(pin "2")
